Commit message: Change launch file and start to tune P3020

File: dsr_description2/ros2_control/p3020.mj_ros2_control.xacro (robot description, xacro)
@@ -4,5 +4,5 @@
     <xacro:include filename="$(find dsr_description2)/config/macro.transmission.xacro" />
     <xacro:include filename="$(find dsr_description2)/config/macro.materials.xacro" />
-    <xacro:property name="default_position_kp" value="2500" />
+    <xacro:property name="default_position_kp" value="10000" />
     <xacro:property name="default_position_ki" value="10" />
     <xacro:property name="default_position_kd" value="10" />
